File: PCB/ISOCHet.kicad_pcb (KiCad board)
At the start: 2 copper layers, 57.1 x 38.1 mm, 19 parts, among them J1 USB_C_Receptacle_USB2.0, J2 Conn_01x08_Pin, SW0 BOOT, SW1 TAB, SW2 ENTER, SW3 CAPS, SW4 CAPS_STEP1.5, SW5 CAPS_STEP1.25, U1 CH552G, U2 USBLC6-2P6

Commit message: Change routing of UDM and UDP
Now leave U2 straight down rather than at 90°
Changed lines of the file:
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@@
   (arc (start 156.475 42.125) (mid 157.182107 42.417893) (end 157.475 43.125) (width 0.25) (layer "B.Cu") (net 9))
   (arc (start 152.9125 42.125) (mid 152.205393 41.832107) (end 151.9125 41.125) (width 0.25) (layer "B.Cu") (net 9))
+  (segment (start 160.02 62.668629) (end 160.02 60.808427) (width 0.25) (layer "B.Cu") (net 11))
+  (segment (start 161.7 57.471573) (end 161.7 56.778427) (width 0.25) (layer "B.Cu") (net 11))
+  (segment (start 159.7 53.121573) (end 159.7 52.85) (width 0.25) (layer "B.Cu") (net 11))
   (segment (start 159.619315 63.400685) (end 159.785686 63.234314) (width 0.25) (layer "B.Cu") (net 11))
+  (segment (start 159.385 66.595) (end 159.385 63.966371) (width 0.25) (layer "B.Cu") (net 11))
+  (segment (start 160.605787 59.394213) (end 161.114214 58.885786) (width 0.25) (layer "B.Cu") (net 11))
   (segment (start 159.385 66.595) (end 159.385 69.8375) (width 0.25) (layer "B.Cu") (net 11))
-  (segment (start 160.605787 59.344213) (end 161.114214 58.835786) (width 0.25) (layer "B.Cu") (net 11))
-  (segment (start 161.7 54.65) (end 161.7 57.421573) (width 0.25) (layer "B.Cu") (net 11))
-  (segment (start 159.385 66.595) (end 159.385 63.966371) (width 0.25) (layer "B.Cu") (net 11))
-  (segment (start 160.02 62.668629) (end 160.02 60.758427) (width 0.25) (layer "B.Cu") (net 11))
+  (segment (start 161.114213 55.364213) (end 160.285786 54.535786) (width 0.25) (layer "B.Cu") (net 11))
+  (arc (start 160.285786 54.535786) (mid 159.852241 53.88694) (end 159.7 53.121573) (width 0.25) (layer "B.Cu") (net 11))
+  (arc (start 159.785686 63.234314) (mid 159.959104 62.974775) (end 160.02 62.668629) (width 0.25) (layer "B.Cu") (net 11))
+  (arc (start 160.02 60.808427) (mid 160.172241 60.04306) (end 160.605787 59.394213) (width 0.25) (layer "B.Cu") (net 11))
   (arc (start 159.385 63.966371) (mid 159.445896 63.660224) (end 159.619315 63.400685) (width 0.25) (layer "B.Cu") (net 11))
-  (arc (start 159.785686 63.234314) (mid 159.959104 62.974775) (end 160.02 62.668629) (width 0.25) (layer "B.Cu") (net 11))
-  (arc (start 160.02 60.758427) (mid 160.172241 59.99306) (end 160.605787 59.344213) (width 0.25) (layer "B.Cu") (net 11))
-  (arc (start 161.7 54.65) (mid 161.172792 53.377208) (end 159.9 52.85) (width 0.25) (layer "B.Cu") (net 11))
-  (arc (start 161.114214 58.835786) (mid 161.547759 58.18694) (end 161.7 57.421573) (width 0.25) (layer "B.Cu") (net 11))
+  (arc (start 161.114213 55.364213) (mid 161.547759 56.01306) (end 161.7 56.778427) (width 0.25) (layer "B.Cu") (net 11))
+  (arc (start 161.7 57.471573) (mid 161.547759 58.23694) (end 161.114214 58.885786) (width 0.25) (layer "B.Cu") (net 11))
   (segment (start 131.95 50.725) (end 131.95 44.525) (width 0.25) (layer "F.Cu") (net 12))
   (segment (start 132.95 53.970584) (end 132.95 68.6625) (width 0.25) (layer "F.Cu") (net 12))
@@
   (segment (start 149.38375 61.595) (end 144.62125 61.595) (width 0.25) (layer "B.Cu") (net 15))
   (segment (start 154.305 61.595) (end 149.38375 61.595) (width 0.25) (layer "B.Cu") (net 15))
-  (segment (start 156.894213 59.344213) (end 156.385786 58.835786) (width 0.25) (layer "B.Cu") (net 16))
-  (segment (start 157.880685 63.400685) (end 157.714314 63.234314) (width 0.25) (layer "B.Cu") (net 16))
-  (segment (start 157.48 62.668629) (end 157.48 60.758427) (width 0.25) (layer "B.Cu") (net 16))
-  (segment (start 155.8 54.65) (end 155.8 57.421573) (width 0.25) (layer "B.Cu") (net 16))
-  (segment (start 158.115 66.595) (end 158.115 63.966371) (width 0.25) (layer "B.Cu") (net 16))
-  (arc (start 156.894213 59.344213) (mid 157.327759 59.99306) (end 157.48 60.758427) (width 0.25) (layer "B.Cu") (net 16))
-  (arc (start 158.115 63.966371) (mid 158.054104 63.660224) (end 157.880685 63.400685) (width 0.25) (layer "B.Cu") (net 16))
-  (arc (start 155.8 54.65) (mid 156.327208 53.377208) (end 157.6 52.85) (width 0.25) (layer "B.Cu") (net 16))
-  (arc (start 157.714314 63.234314) (mid 157.540896 62.974775) (end 157.48 62.668629) (width 0.25) (layer "B.Cu") (net 16))
-  (arc (start 155.8 57.421573) (mid 155.952241 58.18694) (end 156.385786 58.835786) (width 0.25) (layer "B.Cu") (net 16))
+  (segment (start 155.8 56.778427) (end 155.8 57.471573) (width 0.25) (layer "B.Cu") (net 16))
+  (segment (start 157.48 60.808427) (end 157.48 62.668629) (width 0.25) (layer "B.Cu") (net 16))
+  (segment (start 157.214213 54.535787) (end 156.385786 55.364214) (width 0.25) (layer "B.Cu") (net 16))
+  (segment (start 156.385787 58.885787) (end 156.894214 59.394214) (width 0.25) (layer "B.Cu") (net 16))
+  (segment (start 157.8 52.85) (end 157.8 53.121573) (width 0.25) (layer "B.Cu") (net 16))
+  (segment (start 158.115 63.966371) (end 158.115 66.595) (width 0.25) (layer "B.Cu") (net 16))
+  (segment (start 157.714314 63.234314) (end 157.880685 63.400685) (width 0.25) (layer "B.Cu") (net 16))
+  (arc (start 157.48 60.808427) (mid 157.327759 60.04306) (end 156.894214 59.394214) (width 0.25) (layer "B.Cu") (net 16))
+  (arc (start 156.385786 55.364214) (mid 155.952241 56.01306) (end 155.8 56.778427) (width 0.25) (layer "B.Cu") (net 16))
+  (arc (start 157.48 62.668629) (mid 157.540896 62.974775) (end 157.714314 63.234314) (width 0.25) (layer "B.Cu") (net 16))
+  (arc (start 157.880685 63.400685) (mid 158.054104 63.660224) (end 158.115 63.966371) (width 0.25) (layer "B.Cu") (net 16))
+  (arc (start 156.385787 58.885787) (mid 155.952241 58.23694) (end 155.8 57.471573) (width 0.25) (layer "B.Cu") (net 16))
+  (arc (start 157.214213 54.535787) (mid 157.647759 53.88694) (end 157.8 53.121573) (width 0.25) (layer "B.Cu") (net 16))
   (segment (start 135.65 44.525) (end 135.65 50.725) (width 0.25) (layer "F.Cu") (net 17))
   (segment (start 164.25 65.3875) (end 164.25 54.25) (width 0.4) (layer "F.Cu") (net 17))
