File: PCB/ISOCHet.kicad_sch (KiCad schematic)
At the start: 19 parts, among them J1 USB_C_Receptacle_USB2.0, J2 Conn_01x08_Pin, SW0 BOOT, SW1 TAB, SW2 ENTER, SW3 CAPS, SW4 CAPS_STEP1.5, SW5 CAPS_STEP1.25, U1 CH552E, U2 USBLC6-2P6

Commit message: Move R1 & R2 to top of board
Parts:
- R1, R2: footprint Project Library:R_0603_1608Metric_Pad0.98x0.95mm_HandSolder -> Resistor_SMD:R_0603_1608Metric_Pad0.98x0.95mm_HandSolder
Changed lines of the file:
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@@
 			)
 		)
-		(property "Footprint" "Project Library:R_0603_1608Metric_Pad0.98x0.95mm_HandSolder"
+		(property "Footprint" "Resistor_SMD:R_0603_1608Metric_Pad0.98x0.95mm_HandSolder"
 			(at 60.706 47.498 90)
 			(effects
@@
 			)
 		)
-		(property "Footprint" "Project Library:R_0603_1608Metric_Pad0.98x0.95mm_HandSolder"
+		(property "Footprint" "Resistor_SMD:R_0603_1608Metric_Pad0.98x0.95mm_HandSolder"
 			(at 60.706 46.482 90)
 			(effects

Commit message: Fix project symbol library and CH552 symbol names
Parts:
- U1: symbol Project Library:MCU_CM552E_MSOP-10 -> Project Library:MCU_CH552E_MSOP-10
Changed lines of the file:
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@@
 	)
 	(symbol
-		(lib_id "Project Library:MCU_CM552E_MSOP-10")
+		(lib_id "Project Library:MCU_CH552E_MSOP-10")
 		(at 228.6 48.26 0)
 		(unit 1)
